Commit message: Added grav comp code to mujoco controller

File: descriptions/gen3.urdf (robot description, URDF)
Before this commit: robot gen3_arm, 10 links, 9 joints
Links:
- link base_link: geometry collision mesh filename=package://arthur_control/descriptions/meshes/base_link.STL; visual mesh filename=package://arthur_control/descriptions/meshes/base_link.STL
- link bracelet_link: geometry collision mesh filename=package://arthur_control/descriptions/meshes/bracelet_with_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; visual mesh filename=package://arthur_control/descriptions/meshes/bracelet_with_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
- link ee_adapter_link: geometry collision mesh filename=package://arthur_control/descriptions/meshes/ReamerAssembly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; visual mesh filename=package://arthur_control/descriptions/meshes/ReamerAssembly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
- link forearm_link: geometry collision mesh filename=package://arthur_control/descriptions/meshes/forearm_link.S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; visual mesh filename=package://arthur_control/descriptions/meshes/forearm_link.S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
- link half_arm_1_link: geometry collision mesh filename=package://arthur_control/descriptions/meshes/half_arm_1_lin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; visual mesh filename=package://arthur_control/descriptions/meshes/half_arm_1_lin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
- link half_arm_2_link: geometry collision mesh filename=package://arthur_control/descriptions/meshes/half_arm_2_lin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; visual mesh filename=package://arthur_control/descriptions/meshes/half_arm_2_lin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
- link shoulder_link: geometry collision mesh filename=package://arthur_control/descriptions/meshes/shoulder_link.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; visual mesh filename=package://arthur_control/descriptions/meshes/shoulder_link.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
- link spherical_wrist_1_link: geometry collision mesh filename=package://arthur_control/descriptions/meshes/spherical_wris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; visual mesh filename=package://arthur_control/descriptions/meshes/spherical_wris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
- link spherical_wrist_2_link: geometry collision mesh filename=package://arthur_control/descriptions/meshes/spherical_wris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; visual mesh filename=package://arthur_control/descriptions/meshes/spherical_wris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
